File: Circuits/joystick/Joystick.kicad_sch (KiCad schematic)
At the start: 5 parts, among them J1 USB_B_Micro, U1 Sample RF module (HC-12 actua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

Commit message: modified directory name
Other:
- title: (none) -> Joystick
Changed lines of the file:
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@@
 	(generator_version "9.0")
 	(paper "A4")
+	(title_block
+		(title "Joystick")
+	)
 	(junction
 		(at 85.09 26.67)
